File: schematics_and_boards/mini base/mini base.kicad_pcb (KiCad board)
At the start: 4 copper layers, 25.4 x 25.4 mm, 34 parts, among them Q1 Q_Photo_NPN, Q2 Q_Photo_NPN, Q3 Q_Photo_NPN, Q4 Q_Photo_NPN, SW1 JJBV0UG335NONPRTR, U1 MAX32660GTP+, Y1 32.768kHz

Commit message: initial designs for manufacture
Other:
- board text added: "Mini Base V1"
Changed lines of the file:
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@@
   (gr_circle (center 151.565 99.314) (end 164.265 99.314)
     (stroke (width 0.0381) (type default)) (fill none) (layer "Edge.Cuts"))
+  (gr_text "Mini Base V1" (at 155.8 107.8) (layer "B.SilkS")
+    (effects (font (size 0.8128 0.8128) (thickness 0.1524) bold) (justify left bottom mirror))
+  )
   (segment (start 140.565 100.714) (end 140.565 102.846) (width 0.1) (layer "F.Cu") (net 1))
   (segment (start 151.065001 97.3455) (end 151.065001 96.330999) (width 0.1) (layer "F.Cu") (net 1))
