File: schematics_and_boards/mini base/mini base.kicad_sch (KiCad schematic)
At the start: 34 parts, among them Q1 Q_Photo_NPN, Q2 Q_Photo_NPN, Q3 Q_Photo_NPN, Q4 Q_Photo_NPN, SW1 JJBV0UG335NONPRTR, U1 MAX32660GTP+, Y1 32.768kHz

Commit message: bom updated
Parts:
- BT1: Part # (none) -> BC-2600
- C1, C2: Part # (none) -> CL21B105KOFNNNG
- C3, C4: Part # (none) -> CC0805DRNPO9BN6R0
- C5, C6: Part # (none) -> GRM31CR60G227ME11K
- D1, D2, D3, D4: Part # (none) -> VSMB10940
- Q1, Q2, Q3, Q4: Part # (none) -> XZRNI56BF
- R1, R2, R3, R4: Part # (none) -> RMCF0805FT324R
- R5, R6, R7, R8: value R_US -> 20k; Part # (none) -> RMCF0805FT20K0
- R9: Part # (none) -> RMCF0805FT200R
- SW1: Part # (none) -> JJBV0UG335NONPRTR
- U1: Part # (none) -> MAX32660GTP+
- Y1: Part # (none) -> DH2032K76806T1521008
Changed lines of the file:
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@@
+      (effects (font (size 1.27 1.27)) hide)
+    )
+    (property "Part #" "" (at 237.49 121.92 0)
       (effects (font (size 1.27 1.27)) hide)
     )
@@
       (effects (font (size 1.27 1.27)) hide)
     )
+    (property "Part #" "" (at 237.49 132.08 0)
+      (effects (font (size 1.27 1.27)) hide)
+    )
     (pin "1")
     (instances
@@
       (effects (font (size 1.27 1.27)) hide)
     )
+    (property "Part #" "XZRNI56BF" (at 128.27 107.95 0)
+      (effects (font (size 1.27 1.27)) hide)
+    )
     (pin "1")
     (pin "2")
@@
     )
     (property "Datasheet" "~" (at 180.34 66.04 0)
+      (effects (font (size 1.27 1.27)) hide)
+    )
+    (property "Part #" "RMCF0805FT324R" (at 180.34 66.04 0)
       (effects (font (size 1.27 1.27)) hide)
     )
@@
       (effects (font (size 1.27 1.27)) (justify right))
     )
-    (property "Value" "R_US" (at 55.88 123.19 0)
+    (property "Value" "20k" (at 55.88 123.19 0)
       (effects (font (size 1.27 1.27)) (justify right))
     )
@@
       (effects (font (size 1.27 1.27)) hide)
     )
+    (property "Part #" "RMCF0805FT20K0" (at 53.34 121.92 0)
+      (effects (font (size 1.27 1.27)) hide)
+    )
     (pin "1")
     (pin "2")
@@
       (effects (font (size 1.27 1.27)) hide)
     )
+    (property "Part #" "XZRNI56BF" (at 76.2 107.95 0)
+      (effects (font (size 1.27 1.27)) hide)
+    )
     (pin "1")
     (pin "2")
@@
     )
     (property "Datasheet" "https://www.te.com/commerce/DocumentDelivery/DDEController?Action=srchrtrv&DocNm=2331378-1&DocType=DS&DocLang=English" (at 215.9 22.86 0)
+      (effects (font (size 1.27 1.27)) hide)
+    )
+    (property "Part #" "JJBV0UG335NONPRTR" (at 215.9 27.94 0)
       (effects (font (size 1.27 1.27)) hide)
     )
@@
       (effects (font (size 1.27 1.27)) hide)
     )
+    (property "Part #" "" (at 237.49 116.84 0)
+      (effects (font (size 1.27 1.27)) hide)
+    )
     (pin "1")
     (instances
@@
       (effects (font (size 1.27 1.27)) hide)
     )
+    (property "Part #" "RMCF0805FT324R" (at 180.34 43.18 0)
+      (effects (font (size 1.27 1.27)) hide)
+    )
     (pin "1")
     (pin "2")
@@
       (effects (font (size 1.27 1.27)) hide)
     )
+    (property "Part #" "DH2032K76806T1521008" (at 40.64 48.26 0)
+      (effects (font (size 1.27 1.27)) hide)
+    )
     (pin "1")
     (pin "2")
@@
       (effects (font (size 1.27 1.27)) hide)
     )
+    (property "Part #" "XZRNI56BF" (at 50.8 107.95 0)
+      (effects (font (size 1.27 1.27)) hide)
+    )
     (pin "1")
     (pin "2")
@@
       (effects (font (size 1.27 1.27)) hide)
     )
+    (property "Part #" "RMCF0805FT200R" (at 236.22 27.94 0)
+      (effects (font (size 1.27 1.27)) hide)
+    )
     (pin "1")
     (pin "2")
@@
       (effects (font (size 1.27 1.27)) hide)
     )
+    (property "Part #" "" (at 237.49 106.68 0)
+      (effects (font (size 1.27 1.27)) hide)
+    )
     (pin "1")
     (instances
@@
     (property "MANUFACTURER" "VISHAY" (at 165.1 31.75 0)
       (effects (font (size 1.27 1.27)) (justify bottom) hide)
+    )
+    (property "Part #" "VSMB10940" (at 165.1 31.75 0)
+      (effects (font (size 1.27 1.27)) hide)
     )
     (pin "A")
@@
       (effects (font (size 1.27 1.27)) (justify right))
     )
-    (property "Value" "R_US" (at 81.28 123.19 0)
+    (property "Value" "20k" (at 81.28 123.19 0)
       (effects (font (size 1.27 1.27)) (justify right))
     )
@@
       (effects (font (size 1.27 1.27)) hide)
     )
+    (property "Part #" "RMCF0805FT20K0" (at 78.74 121.92 0)
+      (effects (font (size 1.27 1.27)) hide)
+    )
     (pin "1")
     (pin "2")
@@
       (effects (font (size 1.27 1.27)) hide)
     )
+    (property "Part #" "" (at 237.49 111.76 0)
+      (effects (font (size 1.27 1.27)) hide)
+    )
     (pin "1")
     (instances
@@
     )
     (property "Datasheet" "~" (at 237.49 132.08 0)
+      (effects (font (size 1.27 1.27)) hide)
+    )
+    (property "Part #" "" (at 237.49 127 0)
       (effects (font (size 1.27 1.27)) hide)
     )
@@
     (property "Datasheet" "https://www.analog.com/media/en/technical-documentation/data-sheets/max32660.pdf" (at 80.01 27.94 0)
       (effects (font (size 1.27 1.27) italic) hide)
+    )
+    (property "Part #" "MAX32660GTP+" (at 80.01 27.94 0)
+      (effects (font (size 1.27 1.27)) hide)
     )
     (pin "1")
@@
       (effects (font (size 1.27 1.27)) (justify bottom) hide)
     )
+    (property "Part #" "VSMB10940" (at 165.1 43.18 0)
+      (effects (font (size 1.27 1.27)) hide)
+    )
     (pin "A")
     (pin "C")
@@
       (effects (font (size 1.27 1.27)) hide)
     )
+    (property "Part #" "CC0805DRNPO9BN6R0" (at 50.8 52.07 0)
+      (effects (font (size 1.27 1.27)) hide)
+    )
     (pin "1")
     (pin "2")
@@
       (effects (font (size 1.27 1.27)) hide)
     )
+    (property "Part #" "XZRNI56BF" (at 101.6 107.95 0)
+      (effects (font (size 1.27 1.27)) hide)
+    )
     (pin "1")
     (pin "2")
@@
       (effects (font (size 1.27 1.27)) hide)
     )
+    (property "Part #" "RMCF0805FT324R" (at 180.34 54.61 0)
+      (effects (font (size 1.27 1.27)) hide)
+    )
     (pin "1")
     (pin "2")
@@
       (effects (font (size 1.27 1.27)) hide)
     )
+    (property "Part #" "BC-2600" (at 204.47 40.64 0)
+      (effects (font (size 1.27 1.27)) hide)
+    )
     (pin "1")
     (pin "2")
@@
       (effects (font (size 1.27 1.27)) hide)
     )
+    (property "Part #" "GRM31CR60G227ME11K" (at 266.7 31.75 0)
+      (effects (font (size 1.27 1.27)) hide)
+    )
     (pin "1")
     (pin "2")
@@
       (effects (font (size 1.27 1.27)) hide)
     )
+    (property "Part #" "CL21B105KOFNNNG" (at 76.2 58.42 0)
+      (effects (font (size 1.27 1.27)) hide)
+    )
     (pin "1")
     (pin "2")
@@
     (property "MANUFACTURER" "VISHAY" (at 165.1 54.61 0)
       (effects (font (size 1.27 1.27)) (justify bottom) hide)
+    )
+    (property "Part #" "VSMB10940" (at 165.1 54.61 0)
+      (effects (font (size 1.27 1.27)) hide)
     )
     (pin "A")
@@
       (effects (font (size 1.27 1.27)) hide)
     )
+    (property "Part #" "RMCF0805FT324R" (at 180.34 31.75 0)
+      (effects (font (size 1.27 1.27)) hide)
+    )
     (pin "1")
     (pin "2")
@@
       (effects (font (size 1.27 1.27)) hide)
     )
+    (property "Part #" "CC0805DRNPO9BN6R0" (at 27.94 52.07 0)
+      (effects (font (size 1.27 1.27)) hide)
+    )
     (pin "1")
     (pin "2")
@@
       (effects (font (size 1.27 1.27)) hide)
     )
+    (property "Part #" "CL21B105KOFNNNG" (at 64.77 52.07 0)
+      (effects (font (size 1.27 1.27)) hide)
+    )
     (pin "1")
     (pin "2")
@@
     )
     (property "Datasheet" "~" (at 254 31.75 0)
+      (effects (font (size 1.27 1.27)) hide)
+    )
+    (property "Part #" "GRM31CR60G227ME11K" (at 254 31.75 0)
       (effects (font (size 1.27 1.27)) hide)
     )
@@
       (effects (font (size 1.27 1.27)) (justify right))
     )
-    (property "Value" "R_US" (at 106.68 123.19 0)
+    (property "Value" "20k" (at 106.68 123.19 0)
       (effects (font (size 1.27 1.27)) (justify right))
     )
@@
       (effects (font (size 1.27 1.27)) hide)
     )
+    (property "Part #" "RMCF0805FT20K0" (at 104.14 121.92 0)
+      (effects (font (size 1.27 1.27)) hide)
+    )
     (pin "1")
     (pin "2")
@@
       (effects (font (size 1.27 1.27)) hide)
     )
+    (property "Part #" "" (at 237.49 137.16 0)
+      (effects (font (size 1.27 1.27)) hide)
+    )
     (pin "1")
     (instances
@@
     (property "MANUFACTURER" "VISHAY" (at 165.1 66.04 0)
       (effects (font (size 1.27 1.27)) (justify bottom) hide)
+    )
+    (property "Part #" "VSMB10940" (at 165.1 66.04 0)
+      (effects (font (size 1.27 1.27)) hide)
     )
     (pin "A")
@@
       (effects (font (size 1.27 1.27)) (justify right))
     )
-    (property "Value" "R_US" (at 133.35 123.19 0)
+    (property "Value" "20k" (at 133.35 123.19 0)
       (effects (font (size 1.27 1.27)) (justify right))
     )
@@
       (effects (font (size 1.27 1.27)) hide)
     )
+    (property "Part #" "RMCF0805FT20K0" (at 130.81 121.92 0)
+      (effects (font (size 1.27 1.27)) hide)
+    )
